File: samdNano.kicad_pcb (KiCad board)
At the start: 2 copper layers, 50.8 x 17.8 mm, 34 parts, among them J1 Analog, J2 Digital, J3 USB-C, J4 J Link, SW1 RESET, U1 AMS1117-3.3, U2 ATSAMD21G18A-A, Y1 32.768 kHz

Commit message: commit
Connections:
- J1 pad 15: +3V3 -> +3.3V
- J1 pad 2: +3V3 -> +3.3V
- J2 pad 14: DO -> D0
- U2 pad 10: unconnected-(U2-PA05-Pad10) -> A4
Routing:
- net RST: track 0.00 -> 52.0 mm, vias 0 -> 3
- net +3.3V: track 8.28 -> 51.6 mm, vias 0 -> 3
- net D8: track 0.00 -> 36.0 mm, vias 0 -> 1
- net D13: track 0.00 -> 34.3 mm
- net D12: track 0.00 -> 33.5 mm, vias 0 -> 1
- net D9: track 0.00 -> 33.4 mm, vias 0 -> 1
- net D-: track 0.00 -> 33.2 mm
- net D+: track 0.00 -> 32.0 mm, vias 0 -> 2
- net D11: track 0.00 -> 30.6 mm, vias 0 -> 1
- net D10: track 0.00 -> 28.7 mm, vias 0 -> 1
- net D3: track 0.00 -> 27.1 mm, vias 0 -> 1
- net D1: track 0.00 -> 25.1 mm, vias 0 -> 1
- net D2: track 0.00 -> 22.7 mm, vias 0 -> 3
- net A0: track 0.00 -> 22.5 mm, vias 0 -> 1
- net AREF: track 0.00 -> 22.3 mm, vias 0 -> 1
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
Commit message: commit
Parts:
- moved C2 0.39 mm to (123.2, 94.5)
Routing:
- net GND: track 19.0 -> 85.9 mm, vias 6 -> 11
- net +3.3V: track 51.6 -> 87.6 mm, vias 3 -> 5
- net D4: track 0.00 -> 30.0 mm, vias 0 -> 6
- net +5V: track 29.2 -> 47.5 mm, vias 0 -> 2
- net D8: track 36.0 -> 31.6 mm
- net A0: track 22.5 -> 24.5 mm
- net A1: track 17.7 -> 19.7 mm
- net A3: track 8.63 -> 10.0 mm
- net RST: track 52.0 -> 53.1 mm
- net A2: track 16.5 -> 17.6 mm
- net Net-(JP1-A): track 16.8 -> 17.6 mm
- net D5: track 19.8 -> 19.1 mm
- net D3: track 27.1 -> 26.4 mm
- net D-: track 33.2 -> 33.9 mm
- net AREF: track 22.3 -> 22.9 mm
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