File: samdNano.kicad_pcb (KiCad board)
At the start: 2 copper layers, 51.2 x 19.1 mm, 34 parts, among them J1 Analog, J2 Digital, J3 USB-C, J4 J Link, SW1 RESET, U1 AMS1117-3.3, U2 ATSAMD21G18A-A, Y1 32.768 kHz

Commit message: almost finished board
Parts:
- moved R4 2.30 mm to (137.1, 92.6)
- renumbered C11 to C10, C6 to C2, C4 to C3, C3 to C4, C8 to C5, C9 to C6, C2 to C7, C5 to C8, C10 to C9, D2 to D1, D1 to D2, J4 to J1, J3 to J2, J2 to J3, J1 to J4, JP4 to JP2, MH2 to MH1, MH3 to MH2, MH1 to MH3, R3 to R1, R5 to R3, R1 to R4, R4 to R5, R7 to R6, R6 to R7
Connections:
- J4 pad 15: +3.3V -> +5V
Routing:
- net +5V: track 47.5 -> 56.6 mm
- net +3.3V: track 131.8 -> 123.3 mm
- net GND: track 132.8 -> 134.7 mm, vias 13 -> 12
- net D13: track 35.8 -> 35.3 mm
Other:
- board text added: "3.3V"
- board text added: "A0"
- board text added: "A1"
- board text added: "A2"
- board text added: "A3"
- board text added: "A4"
- board text added: "A5"
- board text added: "AREF"
- board text added: "CS"
- board text added: "D0"
- board text added: "D1"
- board text added: "D10"
- board text added: "D11"
- board text added: "D12"
- board text added: "D13"
- board text added: "D2"
- board text added: "D3"
- board text added: "D4"
- board text added: "D5"
- board text added: "D6"
- board text added: "D7"
- board text added: "D8"
- board text added: "D9"
- board text added: "GND"
- board text added: "MISO"
- board text added: "MOSI"
- board text added: "NC"
- board text added: "RST"
- board text added: "SCK"
- board text added: "SCL"
- board text added: "SDA"
- board text added: "VIN"
- board text added: "samdNano+"
- board text added: "v1.0"
