File: samdNano.kicad_sch (KiCad schematic)
At the start: 28 parts, among them J1 Analog, J2 Digital, J3 USB-C, SW1 RESET, U1 AMS1117-3.3, U2 ATSAMD21G18A-A, Y1 32.768 kHz

Commit message: Footprints
Parts:
- removed C12, C7: 100 nF, Capacitor_SMD:C_0805_2012Metric_Pad1.18x1.45mm_HandSolder, symbol Device:C_Small
- removed C14: 100 nF, symbol Device:C_Small
- added C2, C3, C5: 100 nF, Capacitor_SMD:C_0402_1005Metric, symbol Device:C_Small
- added J4: J Link, Connector_PinHeader_1.27mm:PinHeader_2x05_P1.27mm_Vertical_SMD, symbol Connector_Generic:Conn_02x05_Odd_Even
- C1, C4: footprint Capacitor_SMD:C_0805_2012Metric_Pad1.18x1.45mm_HandSolder -> Capacitor_SMD:C_0402_1005Metric; LCSC (none) -> C1525
- C10, C11: footprint (none) -> Capacitor_SMD:C_0805_2012Metric; LCSC (none) -> C15850
- C6: footprint Capacitor_SMD:C_0805_2012Metric_Pad1.18x1.45mm_HandSolder -> Capacitor_SMD:C_0603_1608Metric; LCSC (none) -> C15849
- C8, C9: footprint Capacitor_SMD:C_0805_2012Metric_Pad1.18x1.45mm_HandSolder -> Capacitor_SMD:C_0402_1005Metric; LCSC (none) -> C1555
- D1: footprint LED_SMD:LED_0805_2012Metric_Pad1.15x1.40mm_HandSolder -> LED_SMD:LED_0603_1608Metric; LCSC (none) -> C72038
- D2: footprint LED_SMD:LED_0805_2012Metric_Pad1.15x1.40mm_HandSolder -> LED_SMD:LED_0805_2012Metric; LCSC (none) -> C84256
- J2: footprint Connector_PinHeader_2.54mm:PinHeader_1x15_P2.54mm_Vertical -> Connector_PinHeader_2.54mm:PinHeader_1x18_P2.54mm_Vertical
- J3: LCSC (none) -> C136423
- R1: footprint Resistor_SMD:R_0805_2012Metric_Pad1.20x1.40mm_HandSolder -> Resistor_SMD:R_0402_1005Metric; LCSC (none) -> C25091
- R2, R3: footprint Resistor_SMD:R_0805_2012Metric_Pad1.20x1.40mm_HandSolder -> Resistor_SMD:R_0603_1608Metric; LCSC (none) -> C4177
- R4, R5: footprint Resistor_SMD:R_0805_2012Metric_Pad1.20x1.40mm_HandSolder -> Resistor_SMD:R_0402_1005Metric; LCSC (none) -> C25905
- R6, R7: footprint Resistor_SMD:R_0805_2012Metric_Pad1.20x1.40mm_HandSolder -> Resistor_SMD:R_0402_1005Metric; LCSC (none) -> C11702
- SW1: LCSC (none) -> C2888954
- U2: LCSC (none) -> C78624
Connections:
- net +3.3V: now also R3.2, C2.1, C3.2, C5.1, J4.1 (Pin_1); no longer C4.2, R3.1
- net +5V: now also C4.1
- net A0: now also U2.3 (PA02)
- net A1: now also U2.7 (PB08)
- net A2: now also U2.8 (PB09)
- net A3: now also U2.9 (PA04)
- net A4: now also R3.1; no longer R3.2
- net A5: now also U2.47 (PB02)
- net AREF: now also U2.4 (PA03)
- net D+: now also U2.34 (PA25)
- net D-: now also U2.33 (PA24)
- net D1: now also U2.15 (PA10)
- net D10: now also U2.27 (PA18)
- net D11: now also U2.25 (PA16)
- net D12: now also U2.28 (PA19)
- net D13: now also U2.26 (PA17)
- net D2: now also U2.23 (PA14)
- net D3: now also U2.14 (PA09)
- net D4: now also U2.13 (PA08)
- net D5: now also U2.24 (PA15)
- net D6: now also U2.29 (PA20)
- net D7: now also U2.30 (PA21)
- net D8: now also U2.11 (PA06)
- net D9: now also U2.12 (PA07)
- net GND: now also C4.2, C2.2, C3.1, C5.2, J4.3 (Pin_3), J4.5 (Pin_5); no longer C4.1
- net RST: now also U2.40 (~{RESET}), J4.10 (Pin_10)
- net XIN: now also U2.1 (PA00)
- net XOUT: now also U2.2 (PA01)
- net D0: now reaches U2.16 (PA11)
- net MOSI: now reaches U2.19 (PB10)
- net SCK: now reaches U2.20 (PB11)
- net MISO: now reaches U2.21 (PA12)
- net CS: now reaches U2.22 (PA13)
- net SDA: now reaches U2.31 (PA22)
- net SCL: now reaches U2.32 (PA23)
- net SWCLK: now reaches U2.45 (PA30)
- net SWCLK: now also J4.4 (Pin_4)
- net SWDIO: now reaches U2.46 (PA31)
- net SWDIO: now also J4.2 (Pin_2)
Other:
- note added: "J Link"
- moved on the sheet: C11

Commit message: Basic layout
Parts:
- J1: footprint Connector_PinHeader_2.54mm:PinHeader_1x15_P2.54mm_Vertical -> Connector_PinHeader_2.54mm:PinHeader_1x18_P2.54mm_Vertical; symbol Connector_Generic:Conn_01x15 -> Connector_Generic:Conn_01x18
- J2: symbol Connector_Generic:Conn_01x15 -> Connector_Generic:Conn_01x18
- Y1: footprint Crystal:Crystal_C26-LF_D2.1mm_L6.5mm_Horizontal -> CM7V-T1A-32.768K-12.5PF-20PPM-TA-QA:XTAL_CM7V-T1A-32.768K-12.5PF-20PPM-TA-QA; LCSC (none) -> C32346
Connections:
- net A4: no longer R3.1
- net A5: no longer R2.1
- net CS: now also J2.18 (Pin_18)
- net MISO: now also J1.18 (Pin_18)
- net MOSI: now also J1.17 (Pin_17)
- net SCK: now also J1.16 (Pin_16)
- net SCL: now also J2.17 (Pin_17), R2.1
- net SDA: now also J2.16 (Pin_16), R3.1
Changed lines of the file:
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@@
 	(wire
 		(pts
-			(xy 26.67 59.69) (xy 26.67 64.77)
+			(xy 24.13 59.69) (xy 24.13 64.77)
 		)
 		(stroke
@@
 	(wire
 		(pts
-			(xy 35.56 59.69) (xy 26.67 59.69)
+			(xy 35.56 59.69) (xy 24.13 59.69)
 		)
 		(stroke
@@
 		)
 	)
-	(global_label "A4"
+	(global_label "SDA"
 		(shape input)
 		(at 161.29 137.16 270)
@@
 		)
 		(property "Intersheetrefs" "${INTERSHEET_REFS}"
-			(at 161.29 142.4433 90)
+			(at 161.29 143.7133 90)
 			(effects
 				(font
@@
 		)
 	)
+	(global_label "SDA"
+		(shape input)
+		(at 55.88 64.77 0)
+		(fields_autoplaced yes)
+		(effects
+			(font
+				(size 1.27 1.27)
+			)
+			(justify left)
+		)
+		(property "Intersheetrefs" "${INTERSHEET_REFS}"
+			(at 62.4333 64.77 0)
+			(effects
+				(font
+					(size 1.27 1.27)
+				)
+				(justify left)
+				(hide yes)
+			)
+		)
+	)
 	(global_label "D1"
 		(shape input)
@@
 		)
 	)
+	(global_label "SCK"
+		(shape input)
+		(at 35.56 64.77 180)
+		(fields_autoplaced yes)
+		(effects
+			(font
+				(size 1.27 1.27)
+			)
+			(justify right)
+		)
+		(property "Intersheetrefs" "${INTERSHEET_REFS}"
+			(at 28.8253 64.77 0)
+			(effects
+				(font
+					(size 1.27 1.27)
+				)
+				(justify right)
+				(hide yes)
+			)
+		)
+	)
+	(global_label "SCL"
+		(shape input)
+		(at 55.88 67.31 0)
+		(fields_autoplaced yes)
+		(effects
+			(font
+				(size 1.27 1.27)
+			)
+			(justify left)
+		)
+		(property "Intersheetrefs" "${INTERSHEET_REFS}"
+			(at 62.3728 67.31 0)
+			(effects
+				(font
+					(size 1.27 1.27)
+				)
+				(justify left)
+				(hide yes)
+			)
+		)
+	)
 	(global_label "SWDIO"
 		(shape input)
@@
 		)
 	)
+	(global_label "MOSI"
+		(shape input)
+		(at 35.56 67.31 180)
+		(fields_autoplaced yes)
+		(effects
+			(font
+				(size 1.27 1.27)
+			)
+			(justify right)
+		)
+		(property "Intersheetrefs" "${INTERSHEET_REFS}"
+			(at 27.9786 67.31 0)
+			(effects
+				(font
+					(size 1.27 1.27)
+				)
+				(justify right)
+				(hide yes)
+			)
+		)
+	)
 	(global_label "D12"
 		(shape input)
@@
 		)
 	)
+	(global_label "CS"
+		(shape input)
+		(at 55.88 69.85 0)
+		(fields_autoplaced yes)
+		(effects
+			(font
+				(size 1.27 1.27)
+			)
+			(justify left)
+		)
+		(property "Intersheetrefs" "${INTERSHEET_REFS}"
+			(at 61.3447 69.85 0)
+			(effects
+				(font
+					(size 1.27 1.27)
+				)
+				(justify left)
+				(hide yes)
+			)
+		)
+	)
+	(global_label "MISO"
+		(shape input)
+		(at 35.56 69.85 180)
+		(fields_autoplaced yes)
+		(effects
+			(font
+				(size 1.27 1.27)
+			)
+			(justify right)
+		)
+		(property "Intersheetrefs" "${INTERSHEET_REFS}"
+			(at 27.9786 69.85 0)
+			(effects
+				(font
+					(size 1.27 1.27)
+				)
+				(justify right)
+				(hide yes)
+			)
+		)
+	)
 	(global_label "D-"
 		(shape input)
@@
 		)
 	)
-	(global_label "A5"
+	(global_label "SCL"
 		(shape input)
 		(at 151.13 137.16 270)
@@
 		)
 		(property "Intersheetrefs" "${INTERSHEET_REFS}"
-			(at 151.13 142.4433 90)
+			(at 151.13 143.6528 90)
 			(effects
 				(font
@@
 	)
 	(symbol
-		(lib_id "Connector_Generic:Conn_01x15")
-		(at 40.64 44.45 0)
+		(lib_id "Connector_Generic:Conn_01x18")
+		(at 40.64 46.99 0)
 		(unit 1)
 		(exclude_from_sim no)
@@
 		(dnp no)
 		(property "Reference" "J1"
-			(at 40.64 24.13 0)
+			(at 39.37 20.32 0)
 			(effects
 				(font
 					(size 1.27 1.27)
 				)
+				(justify left)
 			)
 		)
 		(property "Value" "Analog"
-			(at 40.64 64.77 0)
+			(at 37.465 22.86 0)
 			(effects
 				(font
 					(size 1.27 1.27)
 				)
+				(justify left)
 			)
 		)
-		(property "Footprint" "Connector_PinHeader_2.54mm:PinHeader_1x15_P2.54mm_Vertical"
-			(at 40.64 44.45 0)
+		(property "Footprint" "Connector_PinHeader_2.54mm:PinHeader_1x18_P2.54mm_Vertical"
+			(at 40.64 46.99 0)
 			(effects
 				(font
@@
 		)
 		(property "Datasheet" "~"
-			(at 40.64 44.45 0)
+			(at 40.64 46.99 0)
 			(effects
 				(font
@@
 			)
 		)
-		(property "Description" ""
-			(at 40.64 44.45 0)
+		(property "Description" "Generic connector, single row, 01x18, script generated (kicad-library-utils/schlib/autogen/connector/)"
+			(at 40.64 46.99 0)
 			(effects
 				(font
@@
 		(pin "9"
 		)
+		(pin "16"
+		)
+		(pin "17"
+		)
+		(pin "18"
+		)
 		(instances
 			(project "samdNano"
@@
 	)
 	(symbol
-		(lib_id "Connector_Generic:Conn_01x15")
-		(at 50.8 44.45 0)
+		(lib_id "Connector_Generic:Conn_01x18")
+		(at 50.8 46.99 0)
 		(mirror y)
 		(unit 1)
@@
 		(on_board yes)
 		(dnp no)
+		(fields_autoplaced yes)
 		(property "Reference" "J2"
-			(at 50.8 24.13 0)
+			(at 50.8 20.32 0)
 			(effects
 				(font
@@
 		)
 		(property "Value" "Digital"
-			(at 50.8 64.77 0)
+			(at 50.8 22.86 0)
 			(effects
 				(font
@@
 		)
 		(property "Footprint" "Connector_PinHeader_2.54mm:PinHeader_1x18_P2.54mm_Vertical"
-			(at 50.8 44.45 0)
+			(at 50.8 46.99 0)
 			(effects
 				(font
@@
 		)
 		(property "Datasheet" "~"
-			(at 50.8 44.45 0)
+			(at 50.8 46.99 0)
 			(effects
 				(font
@@
 			)
 		)
-		(property "Description" ""
-			(at 50.8 44.45 0)
+		(property "Description" "Generic connector, single row, 01x18, script generated (kicad-library-utils/schlib/autogen/connector/)"
+			(at 50.8 46.99 0)
 			(effects
 				(font
@@
 		(pin "9"
 		)
+		(pin "16"
+		)
+		(pin "17"
+		)
+		(pin "18"
+		)
 		(instances
 			(project "samdNano"
@@
 			)
 		)
-		(property "Footprint" "Crystal:Crystal_C26-LF_D2.1mm_L6.5mm_Horizontal"
+		(property "Footprint" "CM7V-T1A-32.768K-12.5PF-20PPM-TA-QA:XTAL_CM7V-T1A-32.768K-12.5PF-20PPM-TA-QA"
 			(at 204.47 142.24 0)
 			(effects
@@
 			)
 		)
+		(property "LCSC" "C32346"
+			(at 204.47 142.24 0)
+			(effects
+				(font
+					(size 1.27 1.27)
+				)
+				(hide yes)
+			)
+		)
 		(pin "2"
 		)
@@
 	(symbol
 		(lib_id "power:GND")
-		(at 26.67 64.77 0)
+		(at 24.13 64.77 0)
 		(unit 1)
 		(exclude_from_sim no)
@@
 		(fields_autoplaced yes)
 		(property "Reference" "#PWR0104"
-			(at 26.67 71.12 0)
+			(at 24.13 71.12 0)
 			(effects
 				(font
@@
 		)
 		(property "Value" "GND"
-			(at 26.67 68.58 0)
+			(at 24.13 68.58 0)
 			(effects
 				(font
@@
 		)
 		(property "Footprint" ""
-			(at 26.67 64.77 0)
+			(at 24.13 64.77 0)
 			(effects
 				(font
@@
 		)
 		(property "Datasheet" ""
-			(at 26.67 64.77 0)
+			(at 24.13 64.77 0)
 			(effects
 				(font
@@
 		)
 		(property "Description" ""
-			(at 26.67 64.77 0)
+			(at 24.13 64.77 0)
 			(effects
 				(font

Commit message: routing
Parts:
- added JP1: PWR_EN, Jumper:SolderJumper-2_P1.3mm_Open_RoundedPad1.0x1.5mm, symbol Jumper:SolderJumper_2_Open
Connections:
- net VCC is gone; now on net +3V3: J1.15 (Pin_15)
- net +3.3V: now also JP1.2 (B); no longer C10.1, C5.1, U1.2 (VO)
- new net: C10.1, C5.1, JP1.1 (A), U1.2 (VO)
Other:
- moved on the sheet: C10, C11, C5, U1

Commit message: commit
Connections:
- net +3V3 is gone; now on net +3.3V: J1.15 (Pin_15), J1.2 (Pin_2)
- net DO is gone; now on net D0: J2.14 (Pin_14)
- net A4: now also U2.10 (PA05)
Changed lines of the file:
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@@
 		)
 	)
-	(global_label "DO"
+	(global_label "D0"
 		(shape input)
 		(at 55.88 59.69 0)
@@
 		)
 		(property "Intersheetrefs" "${INTERSHEET_REFS}"
-			(at 61.4657 59.69 0)
+			(at 61.3447 59.69 0)
 			(effects
 				(font
@@
 		)
 	)
+	(global_label "A4"
+		(shape input)
+		(at 77.47 97.79 180)
+		(fields_autoplaced yes)
+		(effects
+			(font
+				(size 1.27 1.27)
+			)
+			(justify right)
+		)
+		(property "Intersheetrefs" "${INTERSHEET_REFS}"
+			(at 72.1867 97.79 0)
+			(effects
+				(font
+					(size 1.27 1.27)
+				)
+				(justify right)
+				(hide yes)
+			)
+		)
+	)
 	(global_label "AREF"
 		(shape input)
@@
 	)
 	(symbol
+		(lib_name "+3.3V_5")
+		(lib_id "power:+3.3V")
+		(at 35.56 62.23 90)
+		(unit 1)
+		(exclude_from_sim no)
+		(in_bom yes)
+		(on_board yes)
+		(dnp no)
+		(property "Reference" "#PWR026"
+			(at 39.37 62.23 0)
+			(effects
+				(font
+					(size 1.27 1.27)
+				)
+				(hide yes)
+			)
+		)
+		(property "Value" "+3.3V"
+			(at 29.21 62.23 90)
+			(effects
+				(font
+					(size 1.27 1.27)
+				)
+			)
+		)
+		(property "Footprint" ""
+			(at 35.56 62.23 0)
+			(effects
+				(font
+					(size 1.27 1.27)
+				)
+				(hide yes)
+			)
+		)
+		(property "Datasheet" ""
+			(at 35.56 62.23 0)
+			(effects
+				(font
+					(size 1.27 1.27)
+				)
+				(hide yes)
+			)
+		)
+		(property "Description" "Power symbol creates a global label with name \"+3.3V\""
+			(at 35.56 62.23 0)
+			(effects
+				(font
+					(size 1.27 1.27)
+				)
+				(hide yes)
+			)
+		)
+		(pin "1"
+		)
+		(instances
+			(project "samdNano"
+				(path "/0d35483a-0b12-46cc-b9f2-896fd6831779"
+					(reference "#PWR026")
+					(unit 1)
+				)
+			)
+		)
+	)
+	(symbol
 		(lib_name "GND_5")
 		(lib_id "power:GND")
@@
 	)
 	(symbol
-		(lib_id "power:+3.3V")
-		(at 35.56 62.23 90)
-		(unit 1)
-		(exclude_from_sim no)
-		(in_bom yes)
-		(on_board yes)
-		(dnp no)
-		(fields_autoplaced yes)
-		(property "Reference" "#PWR025"
-			(at 39.37 62.23 0)
-			(effects
-				(font
-					(size 1.27 1.27)
-				)
-				(hide yes)
-			)
-		)
-		(property "Value" "+3V3"
-			(at 31.75 62.2299 90)
-			(effects
-				(font
-					(size 1.27 1.27)
-				)
-				(justify left)
-			)
-		)
-		(property "Footprint" ""
-			(at 35.56 62.23 0)
-			(effects
-				(font
-					(size 1.27 1.27)
-				)
-				(hide yes)
-			)
-		)
-		(property "Datasheet" ""
-			(at 35.56 62.23 0)
-			(effects
-				(font
-					(size 1.27 1.27)
-				)
-				(hide yes)
-			)
-		)
-		(property "Description" ""
-			(at 35.56 62.23 0)
-			(effects
-				(font
-					(size 1.27 1.27)
-				)
-				(hide yes)
-			)
-		)
-		(pin "1"
-		)
-		(instances
-			(project "samdNano"
-				(path "/0d35483a-0b12-46cc-b9f2-896fd6831779"
-					(reference "#PWR025")
-					(unit 1)
-				)
-			)
-		)
-	)
-	(symbol
 		(lib_id "Device:C_Small")
 		(at 135.89 35.56 0)
@@
 	)
 	(symbol
-		(lib_id "power:+3.3V")
-		(at 26.67 25.4 0)
-		(unit 1)
-		(exclude_from_sim no)
-		(in_bom yes)
-		(on_board yes)
-		(dnp no)
-		(fields_autoplaced yes)
-		(property "Reference" "#PWR0102"
-			(at 26.67 29.21 0)
-			(effects
-				(font
-					(size 1.27 1.27)
-				)
-				(hide yes)
-			)
-		)
-		(property "Value" "+3V3"
-			(at 26.67 20.32 0)
-			(effects
-				(font
-					(size 1.27 1.27)
-				)
-			)
-		)
-		(property "Footprint" ""
-			(at 26.67 25.4 0)
-			(effects
-				(font
-					(size 1.27 1.27)
-				)
-				(hide yes)
-			)
-		)
-		(property "Datasheet" ""
-			(at 26.67 25.4 0)
-			(effects
-				(font
-					(size 1.27 1.27)
-				)
-				(hide yes)
-			)
-		)
-		(property "Description" ""
-			(at 26.67 25.4 0)
-			(effects
-				(font
-					(size 1.27 1.27)
-				)
-				(hide yes)
-			)
-		)
-		(pin "1"
-		)
-		(instances
-			(project "samdNano"
-				(path "/0d35483a-0b12-46cc-b9f2-896fd6831779"
-					(reference "#PWR0102")
-					(unit 1)
-				)
-			)
-		)
-	)
-	(symbol
 		(lib_name "+5V_2")
 		(lib_id "power:+5V")
@@
 					(unit 1)
 				)
+			)
+		)
+	)
+	(symbol
+		(lib_name "+3.3V_6")
+		(lib_id "power:+3.3V")
+		(at 26.67 25.4 0)
+		(unit 1)
+		(exclude_from_sim no)
+		(in_bom yes)
+		(on_board yes)
+		(dnp no)
+		(property "Reference" "#PWR025"
+			(at 26.67 29.21 0)
+			(effects
+				(font
+					(size 1.27 1.27)
+				)
+				(hide yes)
+			)
+		)
+		(property "Value" "+3.3V"
+			(at 26.67 21.844 0)
+			(effects
+				(font
+					(size 1.27 1.27)
+				)
+			)
+		)
+		(property "Footprint" ""
+			(at 26.67 25.4 0)
+			(effects
+				(font
+					(size 1.27 1.27)
+				)
+				(hide yes)
+			)
+		)
+		(property "Datasheet" ""
+			(at 26.67 25.4 0)
+			(effects
+				(font
+					(size 1.27 1.27)
+				)
+				(hide yes)
+			)
+		)
+		(property "Description" "Power symbol creates a global label with name \"+3.3V\""
+			(at 26.67 25.4 0)
+			(effects
+				(font
+					(size 1.27 1.27)
+				)
+				(hide yes)
+			)
+		)
+		(pin "1"
+		)
+		(instances
+			(project "samdNano"
+				(path "/0d35483a-0b12-46cc-b9f2-896fd6831779"
+					(reference "#PWR025")
+					(unit 1)
+				)
