File: _autosave-samdNano.kicad_sch (KiCad schematic)
At the start: 30 parts, among them J1 Analog, J2 Digital, J3 USB-C, J4 J Link, SW1 RESET, U1 AMS1117-3.3, U2 ATSAMD21G18A-A, Y1 32.768 kHz

Commit message: almost finished board
Parts:
- renumbered C11 to C10, C6 to C2, C4 to C3, C3 to C4, C8 to C5, C9 to C6, C2 to C7, C5 to C8, C10 to C9, D2 to D1, D1 to D2, J4 to J1, J3 to J2, J2 to J3, J1 to J4, JP4 to JP2, R3 to R1, R5 to R3, R1 to R4, R4 to R5, R7 to R6, R6 to R7
Changed lines of the file:
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@@
 		(on_board yes)
 		(dnp no)
-		(property "Reference" "J1"
+		(property "Reference" "J4"
 			(at 39.37 20.32 0)
 			(effects
@@
 			(project "samdNano"
 				(path "/0d35483a-0b12-46cc-b9f2-896fd6831779"
-					(reference "J1")
+					(reference "J4")
 					(unit 1)
 				)
@@
 		(dnp no)
 		(fields_autoplaced yes)
-		(property "Reference" "J2"
+		(property "Reference" "J3"
 			(at 50.8 20.32 0)
 			(effects
@@
 			(project "samdNano"
 				(path "/0d35483a-0b12-46cc-b9f2-896fd6831779"
-					(reference "J2")
+					(reference "J3")
 					(unit 1)
 				)
@@
 		(dnp no)
 		(fields_autoplaced yes)
-		(property "Reference" "C4"
+		(property "Reference" "C3"
 			(at 236.22 35.5662 0)
 			(effects
@@
 			(project "samdNano"
 				(path "/0d35483a-0b12-46cc-b9f2-896fd6831779"
-					(reference "C4")
+					(reference "C3")
 					(unit 1)
 				)
@@
 		(dnp no)
 		(fields_autoplaced yes)
-		(property "Reference" "R3"
+		(property "Reference" "R1"
 			(at 163.83 133.3499 0)
 			(effects
@@
 			(project "samdNano"
 				(path "/0d35483a-0b12-46cc-b9f2-896fd6831779"
-					(reference "R3")
+					(reference "R1")
 					(unit 1)
 				)
@@
 		(dnp no)
 		(fields_autoplaced yes)
-		(property "Reference" "R6"
+		(property "Reference" "R7"
 			(at 52.07 125.7299 0)
 			(effects
@@
 			(project "samdNano"
 				(path "/0d35483a-0b12-46cc-b9f2-896fd6831779"
-					(reference "R6")
+					(reference "R7")
 					(unit 1)
 				)
@@
 		(dnp no)
 		(fields_autoplaced yes)
-		(property "Reference" "R7"
+		(property "Reference" "R6"
 			(at 29.21 125.7299 0)
 			(effects
@@
 			(project "samdNano"
 				(path "/0d35483a-0b12-46cc-b9f2-896fd6831779"
-					(reference "R7")
+					(reference "R6")
 					(unit 1)
 				)
@@
 		(dnp no)
 		(fields_autoplaced yes)
-		(property "Reference" "C10"
+		(property "Reference" "C9"
 			(at 138.43 34.2962 0)
 			(effects
@@
 			(project "samdNano"
 				(path "/0d35483a-0b12-46cc-b9f2-896fd6831779"
-					(reference "C10")
+					(reference "C9")
 					(unit 1)
 				)
@@
 		(dnp no)
 		(fields_autoplaced yes)
-		(property "Reference" "D2"
+		(property "Reference" "D1"
 			(at 35.56 133.6674 90)
 			(effects
@@
 			(project "samdNano"
 				(path "/0d35483a-0b12-46cc-b9f2-896fd6831779"
-					(reference "D2")
+					(reference "D1")
 					(unit 1)
 				)
@@
 		(dnp no)
 		(fields_autoplaced yes)
-		(property "Reference" "C2"
+		(property "Reference" "C7"
 			(at 106.6863 67.31 90)
 			(effects
@@
 			(project "samdNano"
 				(path "/0d35483a-0b12-46cc-b9f2-896fd6831779"
-					(reference "C2")
+					(reference "C7")
 					(unit 1)
 				)
@@
 		(dnp no)
 		(fields_autoplaced yes)
-		(property "Reference" "JP4"
+		(property "Reference" "JP2"
 			(at 34.29 119.3799 90)
 			(effects
@@
 			(project "samdNano"
 				(path "/0d35483a-0b12-46cc-b9f2-896fd6831779"
-					(reference "JP4")
+					(reference "JP2")
 					(unit 1)
 				)
@@
 		(dnp no)
 		(fields_autoplaced yes)
-		(property "Reference" "R1"
+		(property "Reference" "R4"
 			(at 135.89 154.9399 0)
 			(effects
@@
 			(project "samdNano"
 				(path "/0d35483a-0b12-46cc-b9f2-896fd6831779"
-					(reference "R1")
+					(reference "R4")
 					(unit 1)
 				)
@@
 		(dnp no)
 		(fields_autoplaced yes)
-		(property "Reference" "C11"
+		(property "Reference" "C10"
 			(at 115.57 34.2962 0)
 			(effects
@@
 			(project "samdNano"
 				(path "/0d35483a-0b12-46cc-b9f2-896fd6831779"
-					(reference "C11")
+					(reference "C10")
 					(unit 1)
 				)
@@
 		(on_board yes)
 		(dnp no)
-		(property "Reference" "J4"
+		(property "Reference" "J1"
 			(at 149.86 85.09 0)
 			(effects
@@
 			(project "samdNano"
 				(path "/0d35483a-0b12-46cc-b9f2-896fd6831779"
-					(reference "J4")
+					(reference "J1")
 					(unit 1)
 				)
@@
 		(dnp no)
 		(fields_autoplaced yes)
-		(property "Reference" "C8"
+		(property "Reference" "C5"
 			(at 201.93 129.5335 0)
 			(effects
@@
 			(project "samdNano"
 				(path "/0d35483a-0b12-46cc-b9f2-896fd6831779"
-					(reference "C8")
+					(reference "C5")
 					(unit 1)
 				)
@@
 		(dnp no)
 		(fields_autoplaced yes)
-		(property "Reference" "J3"
+		(property "Reference" "J2"
 			(at 196.85 26.67 0)
 			(effects
@@
 			(project "samdNano"
 				(path "/0d35483a-0b12-46cc-b9f2-896fd6831779"
-					(reference "J3")
+					(reference "J2")
 					(unit 1)
 				)
@@
 		(dnp no)
 		(fields_autoplaced yes)
-		(property "Reference" "D1"
+		(property "Reference" "D2"
 			(at 58.42 133.6674 90)
 			(effects
@@
 			(project "samdNano"
 				(path "/0d35483a-0b12-46cc-b9f2-896fd6831779"
-					(reference "D1")
+					(reference "D2")
 					(unit 1)
 				)
@@
 		(dnp no)
 		(fields_autoplaced yes)
-		(property "Reference" "R5"
+		(property "Reference" "R3"
 			(at 232.41 48.2599 0)
 			(effects
@@
 			(project "samdNano"
 				(path "/0d35483a-0b12-46cc-b9f2-896fd6831779"
-					(reference "R5")
+					(reference "R3")
 					(unit 1)
 				)
@@
 		(dnp no)
 		(fields_autoplaced yes)
-		(property "Reference" "C3"
+		(property "Reference" "C4"
 			(at 85.0963 55.88 90)
 			(effects
@@
 			(project "samdNano"
 				(path "/0d35483a-0b12-46cc-b9f2-896fd6831779"
-					(reference "C3")
+					(reference "C4")
 					(unit 1)
 				)
@@
 		(dnp no)
 		(fields_autoplaced yes)
-		(property "Reference" "C6"
+		(property "Reference" "C2"
 			(at 85.0836 66.04 90)
 			(effects
@@
 			(project "samdNano"
 				(path "/0d35483a-0b12-46cc-b9f2-896fd6831779"
-					(reference "C6")
+					(reference "C2")
 					(unit 1)
 				)
@@
 		(dnp no)
 		(fields_autoplaced yes)
-		(property "Reference" "C9"
+		(property "Reference" "C6"
 			(at 214.63 129.5335 0)
 			(effects
@@
 			(project "samdNano"
 				(path "/0d35483a-0b12-46cc-b9f2-896fd6831779"
-					(reference "C9")
+					(reference "C6")
 					(unit 1)
 				)
@@
 		(dnp no)
 		(fields_autoplaced yes)
-		(property "Reference" "R4"
+		(property "Reference" "R5"
 			(at 222.25 48.2599 0)
 			(effects
@@
 			(project "samdNano"
 				(path "/0d35483a-0b12-46cc-b9f2-896fd6831779"
-					(reference "R4")
+					(reference "R5")
 					(unit 1)
 				)
@@
 		(dnp no)
 		(fields_autoplaced yes)
-		(property "Reference" "C5"
+		(property "Reference" "C8"
 			(at 149.86 34.2962 0)
 			(effects
@@
 			(project "samdNano"
 				(path "/0d35483a-0b12-46cc-b9f2-896fd6831779"
-					(reference "C5")
+					(reference "C8")
 					(unit 1)
 				)
